File: Kicad/A4092/flash.kicad_sch (KiCad schematic)
At the start: 5 parts, among them U13 SST39SF010/020/040, U14 W25X40CLSN

Commit message: A4092 Schematics Revision C
- Power U5 / 74LVC07 from 3.3V rail
- Use ABOEH for 1OEAB on U4 / 74ABT16543
- Add bypass capacitor C501 for U5 / 74LVC07
- Remove EMI filters and capacitors from SCSI lines. They
  are a net negative for signal integrity
- Remove DIP switch circuit as all options are controlled
  by the CPLD / AutoConfig ROM now.
- Remove parallel flash memory, as SPI works reliably and
  is significantly easier to source.
- Remove all ferrite beads from signal lines, as these were
  populated with 0 Ohm resistors in all Proto devices.
- Mark power connector and 12V capacitor as DNP
Parts:
- removed C1401: 100nF, Capacitor_SMD:C_0603_1608Metric_Pad1.08x0.95mm_HandSolder, symbol Device:C_Small
- removed R13: 1K, Resistor_SMD:R_0603_1608Metric_Pad0.98x0.95mm_HandSolder, symbol Device:R_Small
- removed R1401: 10K, Resistor_SMD:R_0603_1608Metric_Pad0.98x0.95mm_HandSolder, symbol Device:R_Small
- removed U13: SST39SF010/020/040, Package_SO:TSOP-I-32_11.8x8mm_P0.5mm, symbol 39SF010-TSOP:SST39SF010
- removed U14: W25X40CLSN, Package_SO:SOIC-8_3.9x4.9mm_P1.27mm, symbol Memory_Flash:W25X40CLSN
